File: ultimate_pwm_repeater.kicad_sch (KiCad schematic)
At the start: 21 parts, among them J1 POWER, J2 SIGNAL, Q1 IRF3205, Q2 IRF3205, Q3 IRF3205, Q4 IRF3205

Commit message: replaced connectors
Parts:
- J1: footprint TerminalBlock_WAGO:TerminalBlock_WAGO_2601-1104_1x04_P3.50mm_Horizontal -> TerminalBlock:TerminalBlock_Degson_DG65C-B-04P
- J2: footprint TerminalBlock_WAGO:TerminalBlock_WAGO_2601-1102_1x02_P3.50mm_Horizontal -> TerminalBlock_Phoenix:TerminalBlock_Phoenix_MKDS-1,5-2-5.08_1x02_P5.08mm_Horizontal
Changed lines of the file:
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@@
 			)
 		)
-		(property "Footprint" "TerminalBlock_WAGO:TerminalBlock_WAGO_2601-1104_1x04_P3.50mm_Horizontal"
+		(property "Footprint" "TerminalBlock:TerminalBlock_Degson_DG65C-B-04P"
 			(at 63.5 30.48 0)
 			(effects
@@
 			)
 		)
-		(property "Footprint" "TerminalBlock_WAGO:TerminalBlock_WAGO_2601-1102_1x02_P3.50mm_Horizontal"
+		(property "Footprint" "TerminalBlock_Phoenix:TerminalBlock_Phoenix_MKDS-1,5-2-5.08_1x02_P5.08mm_Horizontal"
 			(at 63.5 44.45 0)
 			(effects
